File: pcb/tekskey.kicad_sch (KiCad schematic)
At the start: 128 parts, among them J1 Conn_01x08, J2 Conn_01x08, J3 Conn_01x01_Male, J4 Conn_01x01_Male, J5 Conn_01x01_Male, J6 Conn_01x01_Male, SW0 MX_SW_HS, SW1 MX_SW_HS, SW10 MX_SW_HS, SW11 MX_SW_HS, SW12 MX_SW_HS, SW13 MX_SW_HS, SW14 MX_SW_HS, SW15 MX_SW_HS, SW1B1 MX_SW_HS, SW2 MX_SW_HS, SW20 MX_SW_HS, SW21 MX_SW_HS, SW22 MX_SW_HS, SW23 MX_SW_HS, SW24 MX_SW_HS, SW25 MX_SW_HS, SW2B1 MX_SW_HS, SW3 MX_SW_HS, SW30 MX_SW_HS, SW31 MX_SW_HS, SW32 MX_SW_HS, SW33 MX_SW_HS, SW34 MX_SW_HS, SW35 MX_SW_HS, SW3B1 MX_SW_HS, SW4 MX_SW_HS, SW40 MX_SW_HS, SW41 MX_SW_HS, SW42 MX_SW_HS, SW43 MX_SW_HS, SW44 MX_SW_HS, SW45 MX_SW_HS, SW4B1 MX_SW_HS, SW5 MX_SW_HS, SW50 MX_SW_HS, SW51 MX_SW_HS, SW51B1 MX_SW_HS, SW52 MX_SW_HS, SW53 MX_SW_HS, SW54 MX_SW_HS, SW55 MX_SW_HS, SW55B1 MX_SW_HS, SW5B1 MX_SW_HS

Commit message: order v1
Parts:
- renumbered D31 to D101, D32 to D102, D33 to D103, D34 to D104, D35 to D105, D36 to D106, D1 to D107, D2 to D108, D3 to D109, D4 to D110, D5 to D111, D6 to D112, D7 to D113, D8 to D114, D9 to D115, D10 to D116, D11 to D117, D12 to D118, D14 to D119, D15 to D120, D13 to D121, D16 to D122, D17 to D123, D18 to D124, D19 to D125, D20 to D126, D21 to D127, D22 to D128, D23 to D129, D24 to D130, D25 to D131, D26 to D132, D27 to D133, D28 to D134, D29 to D135, D30 to D136, J1 to J101, J2 to J102, J3 to J103, J4 to J104, J5 to J105, J6 to J106, LED0B1 to LED0B101, LED0 to LED101, LED1 to LED102, LED2 to LED103, LED3 to LED104, LED4 to LED105, LED5 to LED106, LED10 to LED107, LED11 to LED108, LED12 to LED109, LED13 to LED110, LED14 to LED111, LED15 to LED112, LED20 to LED113, LED21 to LED114, LED22 to LED115, LED23 to LED116, LED24 to LED117, LED25 to LED118, LED30 to LED119, LED31 to LED120, LED32 to LED121, LED33 to LED122, LED34 to LED123, LED35 to LED124, LED40 to LED125, LED41 to LED126, LED42 to LED127, LED43 to LED128, LED44 to LED129, LED45 to LED130, LED50 to LED131, LED6 to LED132, LED51 to LED133, LED52 to LED134, LED53 to LED135, LED54 to LED136, LED7 to LED137, LED55 to LED138, LED1B1 to LED1B101, LED2B1 to LED2B101, LED3B1 to LED3B101, LED4B1 to LED4B101, SW0 to SW101, SW1 to SW102, SW2 to SW103, SW3 to SW104, SW4 to SW105, SW5 to SW106, SW10 to SW107, SW11 to SW108, SW12 to SW109, SW13 to SW110, SW14 to SW111, SW15 to SW112, SW20 to SW113, SW21 to SW114, SW22 to SW115, SW23 to SW116, SW24 to SW117, SW25 to SW118, SW30 to SW119, SW31 to SW120, SW32 to SW121, SW33 to SW122, SW34 to SW123, SW35 to SW124, SW40 to SW125, SW41 to SW126, SW42 to SW127, SW43 to SW128, SW44 to SW129, SW45 to SW130, SW50 to SW131, SW51 to SW132, SW52 to SW133, SW53 to SW134, SW54 to SW135, SW55 to SW136, SW1B1 to SW1B101, SW2B1 to SW2B101, SW3B1 to SW3B101, SW4B1 to SW4B101, SW51B1 to SW51B101, SW55B1 to SW55B101, SW5B1 to SW5B101
Other:
- added sheet Num (tekskey-num.kicad_sch)

Commit message: adjustments
Parts:
- added U101: YAAJ_WeAct_BlackPill_Part_Like, Footprints:YAAJ_WeAct_BlackPill_SWD_2, symbol YAAJ_WeAct_BlackPill_Part_Like:YAAJ_WeAct_BlackPill_Part_Like
- renumbered J102 to J101, J101 to J102
Connections:
- net +5V: now also U101.18 (5V), U101.40 (5V)
- net GND: now also U101.19 (GND), U101.39 (GND)
- net LEDIN: now also U101.33 (PA7)
- net col0: now also U101.27 (PA1)
- net col1: now also U101.28 (PA2)
- net col2: now also U101.29 (PA3)
- net col3: now also U101.34 (PB0)
- net col4: now also U101.35 (PB1)
- net col5: now also U101.37 (PB10)
- net row0: now also U101.2 (PB13)
- net row1: now also U101.12 (PB4)
- net row2: now also U101.11 (PB3)
- net row3: now also U101.10 (PA15)
- net row4: now also U101.4 (PB15)
- net row5: now also U101.3 (PB14)
- no-connect marks 1 -> 18
Other:
- moved on the sheet: J101, J102
