File: pcb/tekskey-rounded.kicad_pcb (KiCad board)
At the start: 2 copper layers, 119.1 x 123.8 mm, 128 parts, among them J1 Conn_01x08, J2 Conn_01x08, J3 Conn_01x01_Male, J4 Conn_01x01_Male, J5 Conn_01x01_Male, J6 Conn_01x01_Male, SW0 MX_SW_HS, SW1 MX_SW_HS, SW10 MX_SW_HS, SW11 MX_SW_HS, SW12 MX_SW_HS, SW13 MX_SW_HS, SW14 MX_SW_HS, SW15 MX_SW_HS, SW1B1 MX_SW_HS, SW2 MX_SW_HS, SW20 MX_SW_HS, SW21 MX_SW_HS, SW22 MX_SW_HS, SW23 MX_SW_HS, SW24 MX_SW_HS, SW25 MX_SW_HS, SW2B1 MX_SW_HS, SW3 MX_SW_HS, SW30 MX_SW_HS, SW31 MX_SW_HS, SW32 MX_SW_HS, SW33 MX_SW_HS, SW34 MX_SW_HS, SW35 MX_SW_HS, SW3B1 MX_SW_HS, SW4 MX_SW_HS, SW40 MX_SW_HS, SW41 MX_SW_HS, SW42 MX_SW_HS, SW43 MX_SW_HS, SW44 MX_SW_HS, SW45 MX_SW_HS, SW4B1 MX_SW_HS, SW5 MX_SW_HS, SW50 MX_SW_HS, SW51 MX_SW_HS, SW51B1 MX_SW_HS, SW52 MX_SW_HS, SW53 MX_SW_HS, SW54 MX_SW_HS, SW55 MX_SW_HS, SW55B1 MX_SW_HS, SW5B1 MX_SW_HS

Commit message: add rounded
Routing:
- net col2: track 116.1 -> 112.6 mm
- net col1: track 151.2 -> 147.8 mm
- net col4: track 130.3 -> 127.0 mm
- net row2: track 129.6 -> 132.9 mm
- net col5: track 169.1 -> 166.0 mm
- net row5: track 218.6 -> 216.8 mm
- net col0: track 148.4 -> 146.6 mm
- net Net-(LED40-Pad2): track 26.6 -> 25.4 mm
- net row0: track 104.1 -> 103.1 mm
- net Net-(LED20-Pad2): track 25.6 -> 24.8 mm
- net Net-(LED15-Pad2): track 25.8 -> 25.0 mm
- net Net-(LED35-Pad2): track 26.2 -> 25.5 mm
- net Net-(LED0-Pad2): track 30.9 -> 30.2 mm
